File: HARDWARE/ver1.kicad_sch (KiCad schematic)
At the start: 7 parts

Commit message: Space the EXT headers to fit Olimex Rev B and Rev C, and clean up ERC
The Olimex RP2350-PICO2-XXL moved its EXT headers between revisions:
pin 1 to pin 1 is 23.54mm on Rev A/B and 22.86mm on Rev C. The sockets
were 23.50mm apart, which suits Rev B but leaves a Rev C 0.64mm out -
enough to bend pins. EXT2 now sits at 23.20mm, splitting the difference
so either revision is 0.34mm out. The sockets stay on F.Cu: the Olimex
plugs in face-up from above with its headers on its underside, so both
boards see pin 2 to the left of pin 1 and nothing is mirrored.

Address nets are renamed from the edge-connector pin they sit on (a1-a16)
to the Z80 signal they carry (A15-A0), matching the data nets, which
were already named by signal, and the firmware's PIN_A0 base. The
connections are unchanged.

The four unused edge-connector pins get their signal names - ~{INT} (b2),
~{M1} (b12), ~{HALT} (b14), RESET (b16) - while keeping their
no-connect flags until they're wired to the Pico.

Unused header pins get no-connect flags, and GND gets a PWR_FLAG, since
ground only arrives through connector pins (power comes to the Olimex
over USB) and ERC otherwise reports it undriven. ERC is now clean; DRC
leaves only the deliberate a/b pad renumbering on the XB80 footprint.

Adds a GND pour on both layers, and regenerates the Gerbers, drill
files, PDF and board render.

Co-Authored-By: Claude Opus 5.5 <noreply@anthropic.com>
Connections:
- net A1: now also EXT2.5 (Pin_5), XB80.a15 (Pin_a15); no longer EXT2.37 (Pin_37), XB80.a1 (Pin_a1)
- net A10: now also EXT2.27 (Pin_27), XB80.a6 (Pin_a6); no longer EXT2.15 (Pin_15), XB80.a10 (Pin_a10)
- net A11: now also EXT2.29 (Pin_29), XB80.a5 (Pin_a5); no longer EXT2.13 (Pin_13), XB80.a11 (Pin_a11)
- net A12: now also EXT2.31 (Pin_31), XB80.a4 (Pin_a4); no longer EXT2.11 (Pin_11), XB80.a12 (Pin_a12)
- net A13: now also EXT2.33 (Pin_33), XB80.a3 (Pin_a3); no longer EXT2.9 (Pin_9), XB80.a13 (Pin_a13)
- net A14: now also EXT2.35 (Pin_35), XB80.a2 (Pin_a2); no longer EXT2.7 (Pin_7), XB80.a14 (Pin_a14)
- net A15: now also EXT2.37 (Pin_37), XB80.a1 (Pin_a1); no longer EXT2.5 (Pin_5), XB80.a15 (Pin_a15)
- net A2: now also EXT2.7 (Pin_7), XB80.a14 (Pin_a14); no longer EXT2.35 (Pin_35), XB80.a2 (Pin_a2)
- net A3: now also EXT2.9 (Pin_9), XB80.a13 (Pin_a13); no longer EXT2.33 (Pin_33), XB80.a3 (Pin_a3)
- net A4: now also EXT2.11 (Pin_11), XB80.a12 (Pin_a12); no longer EXT2.31 (Pin_31), XB80.a4 (Pin_a4)
- net A5: now also EXT2.13 (Pin_13), XB80.a11 (Pin_a11); no longer EXT2.29 (Pin_29), XB80.a5 (Pin_a5)
- net A6: now also EXT2.15 (Pin_15), XB80.a10 (Pin_a10); no longer EXT2.27 (Pin_27), XB80.a6 (Pin_a6)
- net A7: now also EXT2.17 (Pin_17), XB80.a9 (Pin_a9); no longer EXT2.25 (Pin_25), XB80.a7 (Pin_a7)
- net A9: now also EXT2.25 (Pin_25), XB80.a7 (Pin_a7); no longer EXT2.17 (Pin_17), XB80.a9 (Pin_a9)
- net GND: now also EXT1.40 (Pin_40), EXT2.39 (Pin_39), EXT2.40 (Pin_40)
- net ~{M1}: now reaches XB80.b12 (Pin_b12)
- net ~{HALT}: now reaches XB80.b14 (Pin_b14)
- net RESET: now reaches XB80.b16 (Pin_b16)
- net ~{INT}: now reaches XB80.b2 (Pin_b2)
- net A16 renamed A0
- no-connect marks 0 -> 52
